File: board/board.kicad_pcb (KiCad board)
At the start: 2 copper layers, 96.5 x 60 mm, 30 parts, among them J2 Barrel_Jack_Switch, Q1 TJ11A10M3, Q2 2SC1815, SW1 SW_Push, SW2 SW_Push, SW3 SW_Push, U1 CC56-12SURKWA

Commit message: rename across project
Other:
- board text added: "Pocket Sunrise PCB v1.0 2024.08.11 yasunori.xyz"
- board text removed: "Artificial Sun PCB v1.0 2024.08.11 yasunori.xyz"
Changed lines of the file:
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@@
 		(layer "Edge.Cuts")
 	)
-	(gr_text "Artificial Sun PCB v1.0\n2024.08.11 yasunori.xyz"
+	(gr_text "Pocket Sunrise PCB v1.0\n2024.08.11 yasunori.xyz"
 		(at 124 145 0)
 		(layer "F.SilkS")
