File: board/board.kicad_sch (KiCad schematic)
At the start: 26 parts, among them J2 Barrel_Jack_Switch, Q1 Q_PMOS_GDS, Q2 Q_NPN_ECB, SW1 SW_Push, SW2 SW_Push, SW3 SW_Push, U1 CC56-12SURKWA

Commit message: rename across project
Other:
- title: Artificial Sun -> Pocket Sunrise
Changed lines of the file:
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@@
 	(paper "A4")
 	(title_block
-		(title "Artificial Sun")
+		(title "Pocket Sunrise")
 		(company "Yasu")
 	)
